Commit message: patching up

File: urdf/env.xacro (robot description, xacro)
@@ -1,5 +1,5 @@
 <?xml version="1.0"?>
 <robot name="env" xmlns:xacro="http://www.ros.org/wiki/xacro">
-<xacro:macro name="env" params="single_arm_setup use_fake_hardware fake_sensor_commands ur_type:='' robot_ip robot_ip_2:=''">
+<xacro:macro name="env" params="single_arm_setup use_fake_hardware fake_sensor_commands ur_type:='' robot_ip robot_ip_2:='' headless_mode:='true'">
   <link name="world"/>
   <link name="start"/>
@@ -40,4 +40,5 @@
       non_blocking_read="true"
       keep_alive_count="10"
+      headless_mode:="${headless_mode}"
       />
     <xacro:env_ur
@@ -54,5 +55,6 @@
       trajectory_port="60004"
       non_blocking_read="true"
-      keep_alive_count="10"/>
+      keep_alive_count="10"
+      headless_mode:="${headless_mode}"/>
   </xacro:unless>
   <xacro:if value="${single_arm_setup}">
@@ -71,5 +73,6 @@
     trajectory_port="60004"
     non_blocking_read="true"
-    keep_alive_count="10"/>
+    keep_alive_count="10"
+    headless_mode:="${headless_mode}"/>
   </xacro:if>
   <!--Joints-->

Commit message: wip

File: urdf/env.xacro (robot description, xacro)
@@ -1,8 +1,30 @@
 <?xml version="1.0"?>
 <robot name="env" xmlns:xacro="http://www.ros.org/wiki/xacro">
-<xacro:macro name="env" params="single_arm_setup use_fake_hardware fake_sensor_commands ur_type:='' robot_ip robot_ip_2:='' headless_mode:='true'">
+<xacro:macro name="env" params="single_arm_setup use_fake_hardware fake_sensor_commands ur_type:='' robot_ip robot_ip_2:='' headless_mode:='false'">
   <link name="world"/>
   <link name="start"/>
   <link name="end"/>
+  <xacro:macro name="cuboid" params="name l w h">
+   <link name="${name}">
+     <visual>
+       <origin xyz="0.0 0.0 ${-h / 2.0}" rpy="0.0 0.0 0.0"/>
+       <geometry>
+         <box size="${l} ${w} ${h}"/>
+       </geometry>
+     </visual>
+     <collision>
+       <origin xyz="0.0 0.0 ${-h / 2.0}" rpy="0.0 0.0 0.0"/>
+       <geometry>
+         <box size="${l} ${w} ${h}"/>
+       </geometry>
+     </collision>
+   </link>
+  </xacro:macro>
+  <xacro:property name="in_m" value="0.0254"/> <!--inches to meters-->
+<!-- Create the two tables -->
+  <xacro:property name="robot_table_l" value="${96 * in_m}"/>
+  <xacro:property name="robot_table_w" value="${72 * in_m}"/>
+  <xacro:property name="robot_table_h" value="${36 * in_m}"/>
+  <xacro:cuboid name="robot_table" l="${robot_table_w}" w="${robot_table_l}" h="${robot_table_h}"/>
   <!--Robot-->
   <xacro:include filename="$(find dual_arm_test)/urdf/ur_macro.xacro"/>
@@ -40,5 +62,5 @@
       non_blocking_read="true"
       keep_alive_count="10"
-      headless_mode:="${headless_mode}"
+      headless_mode="${headless_mode}"
       />
     <xacro:env_ur
@@ -56,5 +78,5 @@
       non_blocking_read="true"
       keep_alive_count="10"
-      headless_mode:="${headless_mode}"/>
+      headless_mode="${headless_mode}"/>
   </xacro:unless>
   <xacro:if value="${single_arm_setup}">
@@ -74,5 +96,5 @@
     non_blocking_read="true"
     keep_alive_count="10"
-    headless_mode:="${headless_mode}"/>
+    headless_mode="${headless_mode}"/>
   </xacro:if>
   <!--Joints-->
@@ -100,9 +122,4 @@
       <origin xyz="0.2 0.1 1.0" rpy="${radians(90)} 0 0"/>
     </joint>
-    <joint name="world_to_obstacle" type="fixed">
-      <parent link="world"/>
-      <child link="obstacle"/>
-      <origin xyz="-0.05 0 1.25" rpy="0 0 0"/>
-    </joint>
   </xacro:unless>
   <joint name="world_to_robot_table" type="fixed">
@@ -111,9 +128,4 @@
     <child link="robot_table"/>
   </joint>
-  <joint name="ABB_object_to_world" type="fixed">
-    <origin xyz="${(-robot_table_w) + (ABB_w / 2) } ${6 * in_m} ${robot_table_h + ABB_h}" rpy="0.0 0.0 0.0"/>
-    <parent link="world"/>
-    <child link="ABB"/>
-  </joint>
 </xacro:macro>
 </robot>

File: urdf/ur_macro.xacro (robot description, xacro)
@@ -46,5 +46,4 @@
       non_blocking_read="${non_blocking_read}"
       keep_alive_count="${keep_alive_count}"
-      headless_mode="${headless_mode}"
       >
       <origin xyz="0 0 0" rpy="0 0 0" />          <!-- position robot in the parent frame -->

Commit message: it's working I'm going to try to not jinx it

File: urdf/env.xacro (robot description, xacro)
@@ -1,5 +1,5 @@
 <?xml version="1.0"?>
 <robot name="env" xmlns:xacro="http://www.ros.org/wiki/xacro">
-<xacro:macro name="env" params="single_arm_setup use_fake_hardware fake_sensor_commands ur_type:='' robot_ip robot_ip_2:='' headless_mode:='false'">
+<xacro:macro name="env" params="single_arm_setup use_fake_hardware fake_sensor_commands ur_type:='' robot_ip computer_ip robot_ip_2:='' headless_mode">
   <link name="world"/>
   <link name="start"/>
@@ -56,4 +56,5 @@
       generate_ros2_control_tag="true"
       robot_ip="${robot_ip}"
+      reverse_ip="${computer_ip}"
       script_command_port="50005"
       reverse_port="50001"
@@ -72,4 +73,5 @@
       generate_ros2_control_tag="true"
       robot_ip="${robot_ip_2}"
+      reverse_ip="${computer_ip}"
       script_command_port="50010"
       reverse_port="50006"
@@ -90,8 +92,9 @@
     joint_limits_file="$(find ur_description)/config/ur5e/joint_limits.yaml"
     robot_ip="${robot_ip}"
-    script_command_port="60005"
-    reverse_port="60001"
-    script_sender_port="60002"
-    trajectory_port="60004"
+    reverse_ip="${computer_ip}"
+    script_command_port="50005"
+    reverse_port="50001"
+    script_sender_port="50002"
+    trajectory_port="50004"
     non_blocking_read="true"
     keep_alive_count="10"

File: urdf/top_level.xacro (robot description, xacro)
@@ -3,7 +3,8 @@
   <xacro:arg name="robot_ip" default="0.0.0.0"/>
   <xacro:arg name="robot_ip_2" default="0.0.0.0"/>
+  <xacro:arg name="computer_ip" default="172.31.1.17"/>
   <xacro:arg name="fake_sensor_commands" default="true"/>
   <xacro:arg name="use_fake_hardware" default="true"/>
-  <xacro:arg name="headless_mode" default="false"/>
+  <xacro:arg name="headless_mode" default="true"/>
   <xacro:arg name="ur_type" default="ur10e"/>
   <xacro:include filename="$(find dual_arm_test)/urdf/env.xacro"/>
@@ -12,4 +13,5 @@
     use_fake_hardware="$(arg use_fake_hardware)"
     robot_ip="$(arg robot_ip)"
+    computer_ip="$(arg computer_ip)"
     robot_ip_2="$(arg robot_ip_2)"
     headless_mode="$(arg headless_mode)"

File: urdf/ur_macro.xacro (robot description, xacro)
@@ -10,4 +10,5 @@
   joint_limits_file:=''
   robot_ip:=''
+  reverse_ip:=''
   script_command_port
   reverse_port
@@ -16,5 +17,5 @@
   non_blocking_read:='true'
   keep_alive_count:='10'
-  headless_mode:='true'"
+  headless_mode"
   >
   <!--Use default joint limits if joint_limits_file param is empty-->
@@ -55,4 +56,5 @@
       tf_prefix="${tf_prefix}"
       robot_ip="${robot_ip}"
+      reverse_ip="${reverse_ip}"
       parent="${parent_link}"
       joint_limits_parameters_file="${joint_limits_params_file}"
